File: routes/routes.kicad_pcb (KiCad board)
At the start: 2 copper layers, 144.6 x 88.9 mm, 24 parts, among them J2 AudioJack4dpb, SW1 SW_Push, SW10 SW_Push, SW11 SW_Push, SW12 SW_Push, SW13 SW_Push, SW14 SW_Push, SW15 SW_Push, SW16 SW_Push, SW17 SW_Push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

Commit message: Routes ok
Parts:
- added ?: , , F.Cu at (151.4, 95.7)
- added G***: LOGO, LOGO, F.Cu at (120.3, 58.5)
- moved ? 0.92 mm to (178.8, 115.0)
Connections:
- SW10 pad 1: Switch13 -> Switch10
- SW11 pad 1: Switch9 -> Switch11
- SW12 pad 1: Switch10 -> Switch12
- SW13 pad 1: Switch11 -> Switch13
- SW14 pad 1: Switch13 -> Switch14
- SW15 pad 1: Switch17 -> Switch15
- SW17 pad 1: Switch15 -> Switch17
- SW5 pad 1: Switch13 -> Switch5
- SW6 pad 1: Switch5 -> Switch6
- SW7 pad 1: Switch6 -> Switch7
- SW8 pad 1: Switch7 -> Switch8
- SW9 pad 1: Switch8 -> Switch9
Routing:
- net Switch10: track 0.00 -> 142.1 mm
- net Switch5: track 0.00 -> 129.9 mm
- net Switch14: track 0.00 -> 128.7 mm
- net Switch9: track 0.00 -> 111.7 mm
- net Switch13: track 0.00 -> 97.6 mm
- net Switch4: track 0.00 -> 92.2 mm
- net Switch17: track 0.00 -> 81.4 mm
- net Switch12: track 0.00 -> 80.8 mm
- net Switch8: track 0.00 -> 73.6 mm
- net Switch3: track 0.00 -> 69.9 mm
- net Switch15: track 0.00 -> 64.8 mm
- net Switch11: track 0.00 -> 61.6 mm
- net Switch16: track 0.00 -> 58.5 mm
- net vcc: track 0.00 -> 51.8 mm
- net reset: track 0.00 -> 49.6 mm
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
Commit message: More curves
Parts:
- added G***: LOGO, LOGO, F.Cu at (50.8, 76.5)
- added G***: LOGO, LOGO, F.Cu at (94.5, 144.3)
- added G***: LOGO, LOGO, F.Cu at (113.9, 158.9)
- added G***: LOGO, LOGO, F.Cu at (101.1, 121.3)
- added G***: LOGO, LOGO, F.Cu at (177.4, 109.3)
- added G***: LOGO, LOGO, F.Cu at (120.2, 58.1)
- added G***: LOGO, LOGO, F.Cu at (96.7, 72.8)
- moved G*** 16.7 mm to (136.9, 60.6), turned to 0 degrees
- moved ? 0.35 mm to (151.1, 95.7)
- moved ? 0.07 mm to (78.7, 118.0)
Routing:
- net Switch16: track 58.5 -> 70.9 mm
- net Switch15: track 64.8 -> 74.2 mm
- net Switch10: track 142.1 -> 146.1 mm
