File: kicad/test_reverse_controller/test_reverse_controller.kicad_pcb (KiCad board)
At the start: 2 copper layers, 144.6 x 88.9 mm, 36 parts, among them J2 AudioJack4dpb, SW1 SW_Push, SW10 SW_Push, SW11 SW_Push, SW12 SW_Push, SW13 SW_Push, SW14 SW_Push, SW15 SW_Push, SW16 SW_Push, SW17 SW_Push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

Commit message: Reversed controller ok + up matrix pins
Routing:
- net reset: track 122.7 -> 128.2 mm
- net Switch18: track 35.0 -> 37.2 mm
