File: kicad/chew_v1/chew_v1.kicad_pcb (KiCad board)
At the start: 2 copper layers, 144.4 x 88.9 mm, 44 parts, among them J2 AudioJack4dpb, SW1 SW_Push, SW10 SW_Push, SW11 SW_Push, SW12 SW_Push, SW13 SW_Push, SW14 SW_Push, SW15 SW_Push, SW16 SW_Push, SW17 SW_Push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

Commit message: Ordered
Parts:
- removed the G*** at (153.4, 110.3)

Commit message: Enlarge pads
Parts:
- added G***: LOGO, LOGO, F.Cu at (63.9, 71.3)
- added G***: LOGO, LOGO, B.Cu at (88.2, 68.0)
- added G***: LOGO, LOGO, B.Cu at (87.5, 61.8)
- moved G*** 102.2 mm to (178.5, 111.2), turned to 120 degrees
