File: kicad/chew_v1/chew_v1.kicad_pcb (KiCad board)
At the start: 2 copper layers, 160.3 x 91.9 mm, 40 parts, among them U1 RP2040_Zero, U2 TRRS

Commit message: Mono prod
Connections:
- S15 pad 1: S15 -> S17
- S17 pad 1: S17 -> S15
Routing:
- net GND: track 147.7 -> 0.00 mm
- net S17: track 0.00 -> 86.0 mm
- net S15: track 0.00 -> 61.7 mm

Commit message: Simplify switch traces
Connections:
- S15 pad 1: S17 -> S15
- S17 pad 1: S15 -> S17
Changed lines of the file:
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@@
 		(fp_arc
 			(start -6.679999 7.000001)
-			(mid -6.902135 6.916276)
+			(mid -6.902134 6.916276)
 			(end -7.000001 6.699999)
 			(stroke
@@
 		(fp_arc
 			(start -6.679999 7.000001)
-			(mid -6.902135 6.916276)
+			(mid -6.902134 6.916276)
 			(end -7.000001 6.699999)
 			(stroke
@@
 			(size 2.6 2.6)
 			(layers "B.Cu" "B.Paste" "B.Mask")
-			(net 16 "S15")
+			(net 18 "S17")
 			(pinfunction "1")
 			(pintype "passive")
@@
 			(size 2.6 2.6)
 			(layers "B.Cu")
-			(net 16 "S15")
+			(net 18 "S17")
 			(pinfunction "1")
 			(pintype "passive")
@@
 			(layers "*.Cu" "*.Mask")
 			(remove_unused_layers no)
-			(net 16 "S15")
+			(net 18 "S17")
 			(pinfunction "1")
 			(pintype "passive")
@@
 			(size 2.6 2.6)
 			(layers "F.Cu" "F.Paste" "F.Mask")
-			(net 16 "S15")
+			(net 18 "S17")
 			(pinfunction "1")
 			(pintype "passive")
@@
 			(size 2.6 2.6)
 			(layers "F.Cu")
-			(net 16 "S15")
+			(net 18 "S17")
 			(pinfunction "1")
 			(pintype "passive")
@@
 			(size 2.6 2.6)
 			(layers "B.Cu" "B.Paste" "B.Mask")
-			(net 18 "S17")
+			(net 16 "S15")
 			(pinfunction "1")
 			(pintype "passive")
@@
 			(size 2.6 2.6)
 			(layers "B.Cu")
-			(net 18 "S17")
+			(net 16 "S15")
 			(pinfunction "1")
 			(pintype "passive")
@@
 			(layers "*.Cu" "*.Mask")
 			(remove_unused_layers no)
-			(net 18 "S17")
+			(net 16 "S15")
 			(pinfunction "1")
 			(pintype "passive")
@@
 			(size 2.6 2.6)
 			(layers "F.Cu" "F.Paste" "F.Mask")
-			(net 18 "S17")
+			(net 16 "S15")
 			(pinfunction "1")
 			(pintype "passive")
@@
 			(size 2.6 2.6)
 			(layers "F.Cu")
-			(net 18 "S17")
+			(net 16 "S15")
 			(pinfunction "1")
 			(pintype "passive")
