File: kicad/chew_v1/chew_v1_backplate.kicad_pcb (KiCad board)
At the start: 2 copper layers, 144.4 x 88.9 mm, 42 parts

Commit message: Up backplates
Parts:
- removed the G*** at (50.2, 91.6)
- removed the G*** at (102.9, 84.3)
- removed the G*** at (171.0, 135.1)
- removed the G*** at (141.4, 129.8)
- removed the G*** at (71.1, 68.5)
- removed the G*** at (143.4, 199.6)
- removed the G*** at (62.2, 117.2)
- removed the G*** at (71.3, 77.7)
- removed the G*** at (137.6, 126.7)
- removed the G*** at (156.8, 101.3)
- removed the G*** at (166.1, 117.7)
- removed the G*** at (85.2, 111.8)
- removed the G*** at (117.0, 83.4)
- removed the G*** at (65.3, 125.0)
- removed the G*** at (156.9, 116.2)
- removed the G*** at (71.1, 74.4)
- removed the G*** at (77.9, 76.5)
- removed the G*** at (156.9, 77.5)
- removed the G*** at (69.9, 109.0)
- removed the G*** at (84.4, 49.5)
- removed the G*** at (132.5, 132.7)
- removed the G*** at (82.7, 159.0)
- removed the G*** at (70.9, 114.1)
- removed the G*** at (95.9, 119.3)
- removed the G*** at (144.9, 66.2)
- removed the G*** at (102.8, 93.7)
- removed the G*** at (62.7, 89.6)
- removed the G*** at (57.2, 105.6)
- removed the G*** at (139.6, 128.1)
- removed the G*** at (153.7, 99.1)
- removed the G*** at (80.8, 72.2)
- removed the G*** at (142.0, 52.4)
- removed the G*** at (114.6, 89.1)
- removed the G*** at (69.5, 123.1)
- removed the G*** at (99.6, 130.1)
- removed the G*** at (108.9, 99.2)
- added G***: LOGO, LOGO, F.Cu at (65.3, 124.6)
- added G***: LOGO, LOGO, F.Cu at (115.4, 92.7)
- added G***: LOGO, LOGO, F.Cu at (109.6, 102.7)
- added G***: LOGO, LOGO, F.Cu at (103.7, 87.8)
- added G***: LOGO, LOGO, F.Cu at (92.0, 130.6)
- added G***: LOGO, LOGO, F.Cu at (153.6, 134.2)
- added G***: LOGO, LOGO, F.Cu at (70.0, 117.5)
- added G***: LOGO, LOGO, F.Cu at (70.3, 73.5)
- added G***: LOGO, LOGO, F.Cu at (98.3, 132.3)
- added G***: LOGO, LOGO, F.Cu at (143.8, 54.9)
- added G***: LOGO, LOGO, B.Cu at (83.5, 47.4)
- added G***: LOGO, LOGO, F.Cu at (76.3, 79.8)
- added G***: LOGO, LOGO, B.Cu at (141.3, 62.9)
- added G***: LOGO, LOGO, B.Cu at (69.0, 128.6)
- added G***: LOGO, LOGO, B.Cu at (116.6, 89.6)
- added G***: LOGO, LOGO, B.Cu at (153.0, 97.9)
- added G***: LOGO, LOGO, B.Cu at (98.6, 94.1)
- added G***: LOGO, LOGO, B.Cu at (51.1, 104.9)
- added G***: LOGO, LOGO, B.Cu at (68.7, 69.1)
- added G***: LOGO, LOGO, B.Cu at (156.1, 114.9)
- added G***: LOGO, LOGO, B.Cu at (68.0, 110.2)
- added G***: LOGO, LOGO, B.Cu at (122.3, 132.4)
- added G***: LOGO, LOGO, F.Cu at (39.3, 98.0)
- added G***: LOGO, LOGO, B.Cu at (163.5, 115.8)
- added G***: LOGO, LOGO, B.Cu at (64.8, 82.4)
- added G***: LOGO, LOGO, B.Cu at (155.0, 78.7)
- added G***: LOGO, LOGO, B.Cu at (135.9, 128.3)
- added G***: LOGO, LOGO, B.Cu at (89.9, 129.9)
- added G***: LOGO, LOGO, F.Cu at (79.9, 114.5)
- added G***: LOGO, LOGO, F.Cu at (136.6, 127.3)
- added G***: LOGO, LOGO, F.Cu at (155.4, 102.1)
- added G***: LOGO, LOGO, F.Cu at (73.5, 123.3)
- added G***: LOGO, LOGO, F.Cu at (66.7, 83.3)
- added G***: LOGO, LOGO, F.Cu at (92.1, 47.8)
- moved ? 10.8 mm to (54.4, 82.7)
- moved ? 6.18 mm to (82.9, 122.3)
- moved REF** 3.80 mm to (108.5, 93.9), turned to -7.5 degrees
- moved ? 0.40 mm to (161.5, 124.4)
Other:
- board size 144.4 x 88.9 mm -> 156.2 x 94.3 mm
