File: kicad/chew_v1/chew_v1_zero.kicad_pcb (KiCad board)
At the start: 2 copper layers, 159.8 x 92 mm, 40 parts, among them J2 AudioJack4dpb, SW1 SW_Push, SW10 SW_Push, SW11 SW_Push, SW12 SW_Push, SW13 SW_Push, SW14 SW_Push, SW15 SW_Push, SW16 SW_Push, SW17 SW_Push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

Commit message: Add routes
Parts:
- removed the ? at (224.7, 95.8)
- removed the ? at (256.8, 43.7)
- removed the ? at (265.1, 63.7)
- removed the ? at (224.8, 93.3)
- removed the ? at (256.8, 46.2)
- removed the ? at (225.0, 90.8)
- removed the ? at (267.2, 64.4)
- removed the ? at (256.8, 48.7)
- removed the ? at (256.8, 51.2)
- removed the ? at (224.6, 98.3)
- removed the RZ1 at (245.2, 95.9)
- added G***: LOGO, LOGO, F.Cu at (128.7, 59.5)
- added G***: LOGO, LOGO, B.Cu at (127.6, 58.8)
- added G***: LOGO, LOGO, B.Cu at (66.6, 112.3)
- added G***: LOGO, LOGO, B.Cu at (68.2, 113.3)
- added G***: LOGO, LOGO, B.Cu at (114.9, 131.4)
- added G***: LOGO, LOGO, B.Cu at (99.0, 124.2)
- added G***: LOGO, LOGO, F.Cu at (185.7, 101.7)
- added G***: LOGO, LOGO, F.Cu at (114.1, 130.2)
- added G***: LOGO, LOGO, F.Cu at (111.3, 57.1)
- added G***: LOGO, LOGO, F.Cu at (64.5, 104.5)
- added G***: LOGO, LOGO, F.Cu at (100.5, 123.9)
- added G***: LOGO, LOGO, B.Cu at (67.8, 113.8)
- added G***: LOGO, LOGO, B.Cu at (107.7, 60.9)
- added G***: LOGO, LOGO, B.Cu at (117.3, 56.5)
- moved ? 3.29 mm to (138.8, 62.6)
- moved SW5 1.34 mm to (41.8, 103.1), turned to 51 degrees
- moved ? 1.20 mm to (141.7, 132.7)
- moved ? 1.16 mm to (50.3, 88.1)
- moved ? 0.97 mm to (184.6, 109.0)
- moved SW10 0.76 mm to (55.0, 113.8), turned to 51 degrees
- moved SW14 0.20 mm to (68.2, 124.5), turned to 51 degrees
- moved ? 0.13 mm to (78.2, 131.8)
Connections:
- ? pad : (no net) -> Switch13
- ? pad : (no net) -> Switch11
- ? pad : (no net) -> Switch14
- ? pad : (no net) -> Switch12
Routing:
- net Switch5: track 0.00 -> 346.6 mm, vias 0 -> 3
- net Switch4: track 0.00 -> 166.2 mm, vias 0 -> 1
- net (no net): track 459.8 -> 294.2 mm, vias 6 -> 0
- net Switch10: track 0.00 -> 160.6 mm, vias 0 -> 1
- net Switch14: track 0.00 -> 144.3 mm, vias 0 -> 1
- net Switch9: track 0.00 -> 135.7 mm, vias 0 -> 1
- net Switch3: track 0.00 -> 99.9 mm
- net Switch8: track 0.00 -> 90.2 mm
- net Switch13: track 0.00 -> 72.1 mm, vias 0 -> 1
- net Switch2: track 0.00 -> 69.0 mm
- net Switch16: track 0.00 -> 65.5 mm
- net Switch15: track 0.00 -> 61.7 mm
- net Switch18: track 0.00 -> 61.5 mm, vias 0 -> 1
- net Switch7: track 0.00 -> 57.7 mm
- net Switch12: track 0.00 -> 51.1 mm, vias 0 -> 1
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Other:
- board size 159.8 x 92 mm -> 160.3 x 91.9 mm
- board text added: "chew zéro 0.1"
- board text removed: "chew v0.1"
