File: kicad/chew_zero_v1/chew_v1_zero.kicad_pcb (KiCad board)
At the start: 2 copper layers, 160.3 x 91.9 mm, 44 parts, among them J2 AudioJack4dpb, SW1 SW_Push, SW10 SW_Push, SW11 SW_Push, SW12 SW_Push, SW13 SW_Push, SW14 SW_Push, SW15 SW_Push, SW16 SW_Push, SW17 SW_Push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

Commit message: Ordered
Routing:
- net Switch10: track 159.5 -> 157.6 mm
Other:
- board text added: "Chew zéro 0.1"
- board text removed: "chew zéro 0.1"
