File: kicad/mono_v2/mono_v2_backplate.kicad_pcb (KiCad board)
At the start: 2 copper layers, 257.1 x 125.2 mm, 12 parts

Commit message: Up backplates with buzzer holes
Parts:
- added ?: , , F.Cu at (148.7, 115.7)
- added ?: , , F.Cu at (154.3, 115.7)
- added ?: , , F.Cu at (143.1, 115.7)
- moved G*** 17.2 mm to (152.0, 84.5)
- moved G*** 7.55 mm to (53.1, 77.3)
- moved G*** 7.55 mm to (69.5, 63.5)
